File: circuit/kicad/awds.kicad_sch (KiCad schematic)
At the start: 35 parts, among them J1 JST-PH-5P-F, J10 JST-PH-2P-F, J11 JST-PH-2P-M, J12 JST-PH-5P-F, J13 JST-PH-5P-M, J14 JST-PH-2P-F, J15 JST-PH-2P-M, J3 JST-PH-2P-F, J4 JST-PH-2P-F, J5 JST-PH-2P-F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

Commit message: Added Program with Components
Parts:
- removed D1: LED_RGB, symbol Device:LED
- removed R2: R-200, symbol Device:R
- added D1: LED_KRGB, symbol Device:LED_KRGB
- added R7, R8: R-220, symbol Device:R
Connections:
- net GND: now also D1.1 (K), D1.4 (BA)
- net at J7.1 (Pin_1), J8.1 (Pin_1), Q1.3 (C)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: now also U3.10 (~{SRCLR})
- net at U1.13 (MTDI/GPIO12/ADC2_CH5): no longer J1.3 (Pin_3)
- net at U1.15 (MTCK/GPIO13/ADC2_CH4): no longer J1.4 (Pin_4)
- net at U1.12 (MTMS/GPIO14/ADC2_CH6): no longer J1.5 (Pin_5)
- net at U1.33 (GPIO21): now also J1.3 (Pin_3)
- net at R1.2, SW3.1: now also U1.30 (GPIO18); no longer U1.31 (GPIO19)
- net at J7.2 (Pin_2), J8.2 (Pin_2), K1.5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: now also U3.13 (~{OE})
- net at U2.2 (SDA): now also U1.31 (GPIO19); no longer U1.30 (GPIO18)
- net at U1.27 (GPIO16): now also R8.2
- net at U1.28 (GPIO17): now also R7.1
- net at U1.36 (GPIO22): now also J1.4 (Pin_4)
- net at U1.37 (GPIO23): now also J1.5 (Pin_5)
- new net: D1.3 (GA), R7.2
- new net: D1.2 (RA), R8.1
Other:
- moved on the sheet: R1, SW3, U1, U2
