File: circuit/kicad/ris.kicad_sch (KiCad schematic)
At the start: 36 parts, among them J1 JST-PH-5P-F, J10 JST-PH-2P-F, J11 JST-PH-2P-M, J12 JST-PH-5P-F, J13 JST-PH-5P-M, J14 JST-PH-2P-F, J15 JST-PH-2P-M, J3 JST-PH-2P-F, J4 JST-PH-2P-F, J5 JST-PH-2P-F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

Commit message: Changed Name to Regulated Irrigation System (RIS)
Other:
- note added: "REGULATED IRRIGATION SYSTEM - CIRCUIT"
- note removed: "AWDS CIRCUIT"
- title: AWDS CIRCUIT -> RIS CIRCUIT
Changed lines of the file:
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@@
 	(paper "A3")
 	(title_block
-		(title "AWDS CIRCUIT")
+		(title "RIS CIRCUIT")
 		(date "12/11/25")
 		(rev "1")
@@
 		)
 	)
-	(text "AWDS CIRCUIT"
+	(text "REGULATED IRRIGATION SYSTEM - CIRCUIT"
 		(exclude_from_sim no)
 		(at 24.384 24.638 0)
