File: circuit/ris_command-module/ris_command-module.kicad_sch (KiCad schematic)
At the start: 15 parts, among them J1 JST-PH-5P-M, J12 JST-PH-5P-F, J13 JST-PH-2P-F, J14 JST-PH-5P-M, J15 JST-PH-2P-M, J3 JST-PH-2P-M, J6 JST-PH-2P-M, SW2 SW_DIP_x01, SW3 SW_DIP_x01, U1 AM2302_DHT22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

Commit message: Updated Circuit with Side Outputs & Mosfets
Parts:
- removed J3: JST-PH-2P-M, Connector_JST:JST_PH_B2B-PH-K_1x02_P2.00mm_Vertical, symbol Connector:Conn_01x02_Pin
- removed SW2: SW_DIP_x01, symbol Switch:SW_DIP_x01
- removed SW3: SW_DIP_x01, socket-headers-2pin:HARWIN_M20-7820242, symbol Switch:SW_DIP_x01
- removed U1: AM2302_DHT22, socket-headers-3pin:HARWIN_M20-7820346, symbol Sensor:AM2302
- added J1: JST-PH-2P-M_5V, Connector_JST:JST_PH_B2B-PH-K_1x02_P2.00mm_Vertical, symbol Connector:Conn_01x02_Pin
- added J3: JST-PH-5P-M_ZS042, B5B-PH-K-S:JST_B5B-PH-K-S, symbol Connector:Conn_01x05_Pin
- added J4: Header-3P-F_DHT22, socket-headers-3pin:HARWIN_M20-7820346, symbol Connector:Conn_01x03_Socket
- added J5: JST-PH-2P-M_5V, symbol Connector:Conn_01x02_Pin
- added SC1: Solar_Cell, symbol Device:Solar_Cell
- added SW1: SW_DIP_x01, socket-headers-2pin:HARWIN_M20-7820242, symbol Switch:SW_DIP_x01
- added U2: charge-controller_5V-4.2V, symbol Regulator_Switching:XL1509-3.3
- added U3: buck-cnv-board_3.7V-12V, symbol Regulator_Switching:XL1509-3.3
- BT1: value battery-12v -> battery-3.7V
- J6: value JST-PH-2P-M -> JST-PH-2P-M_12V
- U4: value buck-cnv-board_12v-3.3v -> buck-cnv-board_3.7V-5V
- renumbered J1 to J2, D1 to L1
Connections:
- net +3.3V: now also J3.2 (Pin_2), J4.2 (Pin_2), SW1.2; no longer U4.3 (VOUT)
- net GND: now also J1.2 (Pin_2), J3.1 (Pin_1), J4.1 (Pin_1); no longer U4.4 (GND)
- net at U4.1 (VIN): now also BT1.1 (+), U2.3 (VOUT), U3.1 (VIN); no longer J6.2 (Pin_2)
- net at BT1.2 (-), U4.2 (GND): now also U2.4 (GND), U3.2 (GND); no longer J6.1 (Pin_1)
- net at J2.3 (Pin_3): now also U6.J3-9 (IO18); no longer U6.J3-8 (IO19)
- net at J2.4 (Pin_4): now also U6.J3-11 (IO17); no longer U6.J3-9 (IO18)
- net at J2.5 (Pin_5): now also U6.J3-12 (IO16); no longer U6.J3-11 (IO17)
- net at U6.J3-3 (IO22): now also J3.4 (Pin_4)
- net +5V: now reaches U6.J2-19 (EXT_5V)
- net +5V: now also J1.1 (Pin_1)
- net at U6.J2-9 (IO25): now also SW1.1
- net at U6.J3-2 (IO23): now also J4.3 (Pin_3)
- net at U6.J3-6 (IO21): now also J3.3 (Pin_3); no longer R1.2
- new net: SC1.1 (+), U2.1 (VIN)
- new net: SC1.2 (-), U2.2 (GND)
- new net: J5.1 (Pin_1), U4.3 (VOUT)
- new net: J5.2 (Pin_2), U4.4 (GND)
- new net: J6.1 (Pin_1), U3.3 (VOUT)
- new net: J6.2 (Pin_2), U3.4 (GND)
- new net: R1.2, U6.J3-8 (IO19)
Other:
- note added: "+12V / 3.3V"
- note removed: "+12V"
- moved on the sheet: J6, L1, R1
